File: kicad/Preliminary_Schematic_A.kicad_pcb (KiCad board)
At the start: 2 copper layers, 55.9 x 36.8 mm, 12 parts, among them J1 Input, M1 Motor_Servo, Q1 NMOS, U1 VL53L4CDV0DH/1

Commit message: Add files via upload
Parts:
- added J2: Load Cell System, Connector_PinHeader_2.54mm:PinHeader_1x04_P2.54mm_Vertical, F.Cu at (171.4, 108.0)
- J1: value Input -> Battery Connection
- moved R5 6.62 mm to (132.3, 90.2), turned to 0 degrees
- moved R3 6.62 mm to (132.3, 101.6), turned to 0 degrees
- moved C1 6.23 mm to (164.1, 96.8)
- moved C2 6.23 mm to (164.1, 91.7)
- moved R2 2.79 mm to (132.6, 108.0), turned to 0 degrees
- moved J1 2.54 mm to (171.4, 92.7)
- moved U1 1.78 mm to (133.3, 117.1)
- moved R4 1.62 mm to (132.3, 95.8), turned to 0 degrees
Connections:
- net Net-(J1-Pin_1) renamed GND
- R2 pad 1: /3.3V_ESP32 -> /3.3V ESP32
- R3 pad 1: /3.3V_ESP32 -> /3.3V ESP32
- R4 pad 1: /3.3V_ESP32 -> /3.3V ESP32
- R5 pad 1: /3.3V_ESP32 -> /3.3V ESP32
Routing:
- net Net-(J2-Pin_4): track 0.00 -> 57.6 mm, vias 0 -> 1
- net Net-(J2-Pin_3): track 0.00 -> 51.5 mm, vias 0 -> 1
- net Net-(J1-Pin_2): track 0.00 -> 42.9 mm
- net Net-(U1-XSHUT): track 0.00 -> 41.9 mm
- net /3.3V ESP32: track 0.00 -> 35.9 mm, vias 0 -> 6
- net Net-(U1-GPIO1): track 0.00 -> 33.9 mm
- net Net-(R1-Pad2): track 0.00 -> 26.5 mm
- net GND: track 0.00 -> 23.9 mm, vias 0 -> 5
- net Net-(Q1-G): track 0.00 -> 7.95 mm
- net Net-(M1-PWM): track 0.00 -> 7.08 mm
- added copper zone on F.Cu, net /3.3V ESP32
- added copper zone on B.Cu, net GND
Other:
- board size 55.9 x 36.8 mm -> 52.1 x 36.8 mm

Commit message: Add files via upload
Parts:
- added D1: GPIO3_LED, Connector_PinHeader_2.54mm:PinHeader_1x02_P2.54mm_Vertical, F.Cu at (164.3, 109.0)
- added R6: 150, 1/8W, Resistor_SMD:R_0805_2012Metric_Pad1.20x1.40mm_HandSolder, F.Cu at (156.7, 111.5)
- added TP1: TP_+5V, TestPoint:TestPoint_THTPad_D2.0mm_Drill1.0mm, F.Cu at (176.3, 90.2)
- added TP10: TP_3.3V, TestPoint:TestPoint_THTPad_D2.0mm_Drill1.0mm, F.Cu at (176.8, 102.6)
- added TP2: TP_GND, TestPoint:TestPoint_THTPad_D2.0mm_Drill1.0mm, F.Cu at (176.5, 96.0)
- added TP3: TP_TOF_SDA, TestPoint:TestPoint_THTPad_D2.0mm_Drill1.0mm, F.Cu at (125.2, 116.1)
- added TP4: TP_TOF_SCL, TestPoint:TestPoint_THTPad_D2.0mm_Drill1.0mm, F.Cu at (125.2, 105.4)
- added TP5: TP_TOF_pin5, TestPoint:TestPoint_THTPad_D2.0mm_Drill1.0mm, F.Cu at (125.2, 93.7)
- added TP6: TP_LC_SDA, TestPoint:TestPoint_THTPad_D2.0mm_Drill1.0mm, F.Cu at (176.8, 110.0)
- added TP7: TP_LC_SCL, TestPoint:TestPoint_THTPad_D2.0mm_Drill1.0mm, F.Cu at (176.8, 118.6)
- added TP8: TP_PWM, TestPoint:TestPoint_THTPad_D2.0mm_Drill1.0mm, F.Cu at (170.2, 125.2)
- added TP9: TP_NMOS_Gate, TestPoint:TestPoint_THTPad_D2.0mm_Drill1.0mm, F.Cu at (161.8, 125.2)
- C1: value 100nF -> 100nF ±10%
- C2: value 4.7 uF -> 4.7 uF ±10%
- Q1: value NMOS -> DMN2075U-7
- R1: value 100 -> 100, 1/4W
- U1: value VL53L4CDV0DH/1 -> TOF
- moved M1 2.29 mm to (166.1, 118.1)
- moved Q1 2.29 mm to (158.5, 118.1)
- moved R1 2.29 mm to (150.9, 118.1)
- moved C1 1.27 mm to (164.1, 98.0)
- moved C2 1.27 mm to (164.1, 93.0)
Connections:
- net Net-(J1-Pin_2) renamed +5V
Routing:
- net Net-(J2-Pin_4): track 57.6 -> 90.6 mm, vias 1 -> 2
- net Net-(J2-Pin_3): track 51.5 -> 78.2 mm, vias 1 -> 2
- net Net-(Q1-G): track 7.95 -> 17.9 mm
- net Net-(M1-PWM): track 7.08 -> 15.9 mm
- net Net-(R1-Pad2): track 26.5 -> 35.0 mm
- net Net-(D1-A): track 0.00 -> 6.62 mm
- net +5V: track 42.9 -> 46.7 mm
- net Net-(U1-XSHUT): track 41.9 -> 45.7 mm
- net GND: track 23.9 -> 20.3 mm, vias 5 -> 4
Other:
- board size 52.1 x 36.8 mm -> 57.7 x 42 mm
- board text added: "Anti-Squirrel Birdwatcher & Feeder ECE 411_Group 7: Rev. 3"

Commit message: Add files via upload
Parts:
- added G***: LOGO, LOGO, F.Cu at (125.7, 124.7)
- TP1: value TP_+5V -> +5V
- TP10: value TP_3.3V -> 3.3V
- TP2: value TP_GND -> GND
- TP3: value TP_TOF_SDA -> TOF_SDA
- TP4: value TP_TOF_SCL -> TOF_SCL
- TP5: value TP_TOF_pin5 -> TOF_pin5
- TP6: value TP_LC_SDA -> LC_SDA
- TP7: value TP_LC_SCL -> LC_SCL
- TP8: value TP_PWM -> PWM
- TP9: value TP_NMOS_Gate -> NMOS_Gate
- moved C1 30.1 mm to (142.8, 119.4)
- moved C2 29.8 mm to (142.8, 113.8)
- moved D1 2.90 mm to (163.6, 106.2)
Routing:
- net GND: track 20.3 -> 18.7 mm, vias 4 -> 5
Other:
- board text added: "Anti-Squirrel Birdwatcher & Feeder ECE 411: Group 7 - Rev. 4"
- board text removed: "Anti-Squirrel Birdwatcher & Feeder ECE 411_Group 7: Rev. 3"

Commit message: Add files via upload
Parts:
- XIAO1: footprint XIAO_:XIAO_QTpy_SMD -> XIAO_:XIAO_QTpy
Routing:
- net Net-(J2-Pin_4): track 90.6 -> 100.0 mm, vias 2 -> 1
- net Net-(J2-Pin_3): track 78.2 -> 84.1 mm
- net /3.3V ESP32: track 35.9 -> 38.8 mm, vias 6 -> 7

Commit message: Add files via upload
Parts:
- added D2: D_Zener, Diode_THT:D_DO-41_SOD81_P7.62mm_Horizontal, F.Cu at (165.6, 97.8)
- added R7: 10k, Resistor_SMD:R_0805_2012Metric_Pad1.20x1.40mm_HandSolder, F.Cu at (164.1, 114.0)
- C1: value 100nF ±10% -> 100nF
- C2: value 4.7 uF ±10% -> 4.7 uF
- M1: value Motor_Servo -> Motor Servo
- Q1: value DMN2075U-7 -> AO3400A; footprint Package_TO_SOT_SMD:SOT-23 -> Package_TO_SOT_SMD:SOT-23-3
- R1: value 100, 1/4W -> 100
- R6: value 150, 1/8W -> 150
- moved C1 6.97 mm to (141.5, 112.5), turned to 0 degrees
- moved C2 4.50 mm to (141.5, 118.1), turned to 0 degrees
- moved R1 2.79 mm to (150.2, 115.4)
- moved D1 2.70 mm to (165.4, 104.1)
- moved G*** 2.54 mm to (123.2, 124.7)
- moved TP3 2.54 mm to (122.7, 116.1)
- moved TP4 2.54 mm to (122.7, 105.4)
- moved TP5 2.54 mm to (122.7, 93.7)
- moved J1 1.52 mm to (173.0, 92.7)
- moved J2 1.52 mm to (173.0, 108.0)
- moved TP1 1.52 mm to (177.8, 90.2)
- moved TP10 1.52 mm to (178.3, 102.6)
- moved TP2 1.52 mm to (178.1, 96.0)
- moved TP6 1.52 mm to (178.3, 110.0)
- moved TP7 1.52 mm to (178.3, 118.6)
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Connections:
- XIAO1 pad 5V: +5V -> Net-(D2-A)
Routing:
- net /3.3V ESP32: track 38.8 -> 60.2 mm, vias 7 -> 9
- net Net-(J2-Pin_3): track 84.1 -> 95.0 mm, vias 2 -> 1
- net Net-(J2-Pin_4): track 100.0 -> 108.9 mm
- net Net-(D2-A): track 0.00 -> 8.52 mm
- net Net-(M1-PWM): track 15.9 -> 23.7 mm
- net Net-(U1-XSHUT): track 45.7 -> 53.4 mm
- net Net-(U1-GPIO1): track 33.9 -> 37.8 mm
- net Net-(R1-Pad2): track 35.0 -> 31.4 mm
- net Net-(D1-A): track 7.02 -> 10.2 mm
- net +5V: track 46.7 -> 45.1 mm
- net Net-(Q1-G): track 17.9 -> 19.0 mm, vias 0 -> 1
Other:
- board size 57.7 x 42 mm -> 62 x 42 mm
- board text added: "Anti-Squirrel Birdwatcher & Feeder ECE 411: Group 7 - Rev. 5 Nov 11, 2024"
- board text removed: "Anti-Squirrel Birdwatcher & Feeder ECE 411: Group 7 - Rev. 4"
