File: kicad/Preliminary_Schematic_A.kicad_sch (KiCad schematic)
At the start: 5 parts, among them M1 Motor_Servo, U2 40PC015G, U3 TSSP58038

Commit message: Add files via upload
Parts:
- removed A1: Adafruit_Feather_HUZZAH32_ESP32, Module:Adafruit_Feather, symbol MCU_Module:Adafruit_Feather_HUZZAH32_ESP32
- removed B1: ArduCam_OV2640_Breakout, symbol symbols:ArduCam_OV2640_Breakout
- removed U2: 40PC015G, symbol Sensor_Pressure:40PC015G
- removed U3: TSSP58038, OptoDevice:Vishay_MINICAST-3Pin, symbol Sensor_Proximity:TSSP58038
- added C1: 100nF, Capacitor_SMD:C_0805_2012Metric_Pad1.18x1.45mm_HandSolder, symbol Device:C
- added C2: 4.7 uF, Capacitor_SMD:C_0805_2012Metric_Pad1.18x1.45mm_HandSolder, symbol Device:C
- added J1: Input, Connector_PinHeader_2.54mm:PinHeader_1x02_P2.54mm_Vertical, symbol Connector:Conn_01x02_Pin
- added Q1: NMOS, symbol Simulation_SPICE:NMOS
- added R1: 100, Resistor_SMD:R_0805_2012Metric_Pad1.20x1.40mm_HandSolder, symbol Device:R
- added R2, R3: 3.6k, Resistor_SMD:R_0805_2012Metric_Pad1.20x1.40mm_HandSolder, symbol Device:R
- added R4, R5: 10k, Resistor_SMD:R_0805_2012Metric_Pad1.20x1.40mm_HandSolder, symbol Device:R
- added U1: VL53L4CDV0DH/1, LGA12_STM, symbol 2024-11-07_06-19-20:VL53L4CDV0DH_1
- added XIAO1: ~, Dev_boards:XIAO_QTpy, symbol XIAO:esp32s3
- M1: footprint (none) -> Connector_PinHeader_2.54mm:PinHeader_1x03_P2.54mm_Vertical
Connections:
- net at M1.1 (PWM): now also Q1.1 (D)
- net +BATT: no longer names the net of M1.2 (+)
- net +BATT: now also J1.2 (Pin_2), XIAO1.5V
- net -BATT: no longer names the net of M1.3 (-)
- net -BATT: now also C1.2, C2.2, J1.1 (Pin_1), Q1.3 (S), U1.12 (GND4), U1.2 (AVSSVCSEL), U1.3 (GND), U1.4 (GN2), U1.6 (GND3), XIAO1.GND
- new net: R2.2, U1.10 (SCL), XIAO1.5
- new net: Q1.2 (G), R1.1
- new net: R5.2, U1.5 (XSHUT), XIAO1.0
- new net: R4.2, U1.7 (GPIO1), XIAO1.1
- new net: R1.2, XIAO1.3
- new net: R3.2, U1.9 (SDA), XIAO1.4
- new net 3.3V ESP32: C1.1, C2.1, U1.1 (AVDDVCSEL), U1.11 (AVDD), XIAO1.3V3
- new net 3.3V_ESP32: R2.1, R3.1, R4.1, R5.1
Other:
- note added: "+5V"
- note added: "ESP32 with camera module"
- note added: "GND"
- note added: "Pull Up Resistors"
- note added: "Time of Flight Sensor"
- moved on the sheet: M1

Commit message: Add files via upload
Parts:
- added J2: Load Cell System, Connector_PinHeader_2.54mm:PinHeader_1x04_P2.54mm_Vertical, symbol Connector:Conn_01x04_Pin
- J1: value Input -> Battery Connection
- Q1: value NMOS -> DMN2075U-7; footprint (none) -> Package_TO_SOT_SMD:SOT-23
- U1: footprint LGA12_STM -> ul_VL53L4CDV0DH-1:time of flight
- XIAO1: footprint Dev_boards:XIAO_QTpy -> XIAO_:XIAO_QTpy_SMD
Connections:
- net 3.3V_ESP32 is gone; now on net 3.3V ESP32: R2.1, R3.1, R4.1, R5.1
- net 3.3V ESP32: now also J2.2 (Pin_2)
- net GND: now reaches C1.2, C2.2, J1.1 (Pin_1), M1.3 (-), Q1.3 (S), U1.12 (GND4), U1.2 (AVSSVCSEL), U1.3 (GND), U1.4 (GN2), U1.6 (GND3), XIAO1.GND
- net GND: now also J2.1 (Pin_1)
- net at R2.2, U1.10 (SCL), XIAO1.5: now also J2.3 (Pin_3)
- net at R3.2, U1.9 (SDA), XIAO1.4: now also J2.4 (Pin_4)
Other:
- note removed: "GND"
- title: Anti-Squirrel Birdwatch Feeder Preliminary Schematic -> Anti-Squirrel Birdwatch Feeder Draft Schematic
- moved on the sheet: C1, C2, J1, M1, Q1, R1, R2, R3, R4, R5, U1, XIAO1

Commit message: Add files via upload
Parts:
- added D1: GPIO3_LED, Connector_PinHeader_2.54mm:PinHeader_1x02_P2.54mm_Vertical, symbol Device:LED
- added R6: 150, 1/8W, Resistor_SMD:R_0805_2012Metric_Pad1.20x1.40mm_HandSolder, symbol Device:R
- added TP1: TP_+5V, TestPoint:TestPoint_THTPad_D2.0mm_Drill1.0mm, symbol Connector:TestPoint
- added TP10: TP_3.3V, TestPoint:TestPoint_THTPad_D2.0mm_Drill1.0mm, symbol Connector:TestPoint
- added TP2: TP_GND, TestPoint:TestPoint_THTPad_D2.0mm_Drill1.0mm, symbol Connector:TestPoint
- added TP3: TP_TOF_SDA, TestPoint:TestPoint_THTPad_D2.0mm_Drill1.0mm, symbol Connector:TestPoint
- added TP4: TP_TOF_SCL, TestPoint:TestPoint_THTPad_D2.0mm_Drill1.0mm, symbol Connector:TestPoint
- added TP5: TP_TOF_pin5, TestPoint:TestPoint_THTPad_D2.0mm_Drill1.0mm, symbol Connector:TestPoint
- added TP6: TP_LC_SDA, TestPoint:TestPoint_THTPad_D2.0mm_Drill1.0mm, symbol Connector:TestPoint
- added TP7: TP_LC_SCL, TestPoint:TestPoint_THTPad_D2.0mm_Drill1.0mm, symbol Connector:TestPoint
- added TP8: TP_PWM, TestPoint:TestPoint_THTPad_D2.0mm_Drill1.0mm, symbol Connector:TestPoint
- added TP9: TP_NMOS_Gate, TestPoint:TestPoint_THTPad_D2.0mm_Drill1.0mm, symbol Connector:TestPoint
- C1: value 100nF -> 100nF ±10%
- C2: value 4.7 uF -> 4.7 uF ±10%
- R1: value 100 -> 100, 1/4W
Connections:
- net 3.3V ESP32: now also TP10.1
- net GND: now also D1.1 (K), TP2.1
- net +5V: now reaches J1.2 (Pin_2), M1.2 (+), XIAO1.5V
- net +5V: now also TP1.1
- net at J2.3 (Pin_3), R2.2, U1.10 (SCL)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: now also TP4.1, TP7.1
- net at M1.1 (PWM), Q1.1 (D): now also TP8.1
- net at Q1.2 (G), R1.1: now also TP9.1
- net at R5.2, U1.5 (XSHUT), XIAO1.0: now also TP5.1
- net at R1.2, XIAO1.3: now also R6.2
- net at J2.4 (Pin_4), R3.2, U1.9 (SDA)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: now also TP3.1, TP6.1
- new net: D1.2 (A), R6.1
- no-connect marks 0 -> 6
Other:
- note added: "1/8W Rated Resistors"
- note added: "3.3V"
- note added: "Bypass Capacitors"
- note added: "Connection to Load Cell"
- note added: "GND"
- note added: "Microcontroller"
- note added: "Motor Control Circuit"
- note added: "NMOS Motor Control Switch"
- note added: "Power Input"
- note added: "Pull Up Resistors for I2C Lines"
- note added: "SCL"
- note added: "SDA"
- note added: "Time of Flight Sensor Block"
- note removed: "+5V"
- note removed: "Pull Up Resistors"
- moved on the sheet: C1, C2, J1, J2, M1, Q1, R1, R2, R3, R4, R5, U1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

Commit message: Add files via upload
Parts:
- TP1: value TP_+5V -> +5V
- TP10: value TP_3.3V -> 3.3V
- TP2: value TP_GND -> GND
- TP3: value TP_TOF_SDA -> TOF_SDA
- TP4: value TP_TOF_SCL -> TOF_SCL
- TP5: value TP_TOF_pin5 -> TOF_pin5
- TP6: value TP_LC_SDA -> LC_SDA
- TP7: value TP_LC_SCL -> LC_SCL
- TP8: value TP_PWM -> PWM
- TP9: value TP_NMOS_Gate -> NMOS_Gate
Changed lines of the file:
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@@
 			)
 		)
-		(property "Value" "TP_TOF_pin5"
+		(property "Value" "TOF_pin5"
 			(at 86.36 42.4179 0)
 			(effects
@@
 			)
 		)
-		(property "Value" "TP_GND"
+		(property "Value" "GND"
 			(at 212.09 102.1079 0)
 			(effects
@@
 			)
 		)
-		(property "Value" "TP_+5V"
+		(property "Value" "+5V"
 			(at 162.56 93.2179 0)
 			(effects
@@
 			)
 		)
-		(property "Value" "TP_LC_SDA"
+		(property "Value" "LC_SDA"
 			(at 158.75 119.8879 0)
 			(effects
@@
 			)
 		)
-		(property "Value" "TP_3.3V"
+		(property "Value" "3.3V"
 			(at 154.94 110.9979 0)
 			(effects
@@
 			)
 		)
-		(property "Value" "TP_TOF_SDA"
+		(property "Value" "TOF_SDA"
 			(at 152.4 80.7719 0)
 			(effects
@@
 			)
 		)
-		(property "Value" "TP_PWM"
+		(property "Value" "PWM"
 			(at 90.17 150.3679 0)
 			(effects
@@
 			)
 		)
-		(property "Value" "TP_NMOS_Gate"
+		(property "Value" "NMOS_Gate"
 			(at 148.59 165.6079 0)
 			(effects
@@
 			)
 		)
-		(property "Value" "TP_LC_SCL"
+		(property "Value" "LC_SCL"
 			(at 158.75 136.6519 0)
 			(effects
@@
 			)
 		)
-		(property "Value" "TP_TOF_SCL"
+		(property "Value" "TOF_SCL"
 			(at 134.62 80.7719 0)
 			(effects

Commit message: Add files via upload
Parts:
- XIAO1: footprint XIAO_:XIAO_QTpy_SMD -> XIAO_:XIAO_QTpy
Changed lines of the file:
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@@
 	(title_block
 		(title "Anti-Squirrel Birdwatch Feeder Draft Schematic")
-		(date "2024-11-17")
+		(date "2024-11-19")
 		(rev "D")
 		(company "Group 7: Annika Boyd, Sal Esmaeil, Mitch Montee, Nate Sjullie, Nitin Suryadevara")
@@
 			)
 		)
-		(property "Footprint" "XIAO_:XIAO_QTpy_SMD"
+		(property "Footprint" "XIAO_:XIAO_QTpy"
 			(at 115.57 97.79 0)
 			(effects

Commit message: Add files via upload
Parts:
- added D2: D_Zener, Diode_THT:D_DO-41_SOD81_P7.62mm_Horizontal, symbol Device:D_Zener
- added R7: 10k, 1/8W, Resistor_SMD:R_0805_2012Metric_Pad1.20x1.40mm_HandSolder, symbol Device:R
- Q1: value DMN2075U-7 -> AO3400A; footprint Package_TO_SOT_SMD:SOT-23 -> Package_TO_SOT_SMD:SOT-23-3
Connections:
- net +5V: now also D2.1 (K), R7.1; no longer XIAO1.5V
- net at M1.1 (PWM), Q1.1 (D), TP8.1: now also R7.2
- new net: D2.2 (A), XIAO1.5V
Other:
- note added: "Vth: 0.8 to 1.5 V"
- moved on the sheet: D1, M1, Q1, R6, TP1, TP8, TP9
